Commit message: scratch

File: ros/description/xl330.urdf.xacro (robot description, xacro)
@@ -1,48 +1,33 @@
 <?xml version="1.0"?>
-<robot xmlns:xacro="http://ros.org/wiki/xacro" name="xl330_robot">
+<robot xmlns:xacro="http://ros.org/wiki/xacro" name="blossom">
   <xacro:property name="radius" value="0.02"/>
   <xacro:property name="length" value="0.05"/>
-  <xacro:property name="mass" value="0.05"/>
+  <!-- Base link -->
   <link name="base_link">
     <visual>
-      <geometry>
-        <cylinder radius="${radius}" length="${length}"/>
-      </geometry>
+      <geometry><cylinder radius="${radius}" length="${length}"/></geometry>
       <origin xyz="0 0 0" rpy="0 0 0"/>
-      <material name="gray">
-        <color rgba="0.6 0.6 0.6 1.0"/>
-      </material>
+      <material name="gray"><color rgba="0.6 0.6 0.6 1"/></material>
     </visual>
-    <collision>
-      <geometry>
-        <cylinder radius="${radius}" length="${length}"/>
-      </geometry>
-    </collision>
-    <inertial>
-      <mass value="${mass}"/>
-      <inertia ixx="1e-5" iyy="1e-5" izz="1e-5" ixy="0" ixz="0" iyz="0"/>
-    </inertial>
   </link>
-  <joint name="base_swivel" type="revolute">
+  <!-- Base joint -->
+  <joint name="base_joint" type="revolute">
     <parent link="base_link"/>
-    <child link="swivel_link"/>
+    <child link="base_joint_link"/>
     <origin xyz="0 0 ${length/2}" rpy="0 0 0"/>
     <axis xyz="0 0 1"/>
     <limit lower="-3.14" upper="3.14" effort="1.0" velocity="1.0"/>
   </joint>
-  <link name="swivel_link">
+  <link name="base_joint_link">
     <visual>
-      <geometry>
-        <box size="0.04 0.04 0.02"/>
-      </geometry>
-      <origin xyz="0 0 0.02" rpy="0 0 0"/>
-      <material name="black">
-        <color rgba="0.0 0.0 0.0 1.0"/>
-      </material>
+      <geometry><box size="0.05 0.05 0.03"/></geometry>
+      <origin xyz="0 0 0.015" rpy="0 0 0"/>
+      <material name="black"><color rgba="0 0 0 1"/></material>
     </visual>
   </link>
-  <xacro:macro name="string_motor" params="name parent xyz">
+  <!-- Head joint macro -->
+  <xacro:macro name="head_joint" params="name xyz">
     <joint name="${name}" type="revolute">
-      <parent link="${parent}"/>
+      <parent link="base_joint_link"/>
       <child link="${name}_link"/>
       <origin xyz="${xyz}" rpy="0 0 0"/>
@@ -52,16 +37,24 @@
     <link name="${name}_link">
       <visual>
-        <geometry>
-          <cylinder radius="0.01" length="0.03"/>
-        </geometry>
+        <geometry><cylinder radius="0.01" length="0.03"/></geometry>
         <origin xyz="0 0 0.015" rpy="0 0 0"/>
-        <material name="red">
-          <color rgba="1 0 0 1"/>
-        </material>
+        <material name="red"><color rgba="1 0 0 1"/></material>
       </visual>
     </link>
   </xacro:macro>
-  <xacro:string_motor name="string_left" parent="swivel_link" xyz="0.05 0 0.02"/>
-  <xacro:string_motor name="string_right" parent="swivel_link" xyz="-0.05 0 0.02"/>
-  <xacro:string_motor name="string_back" parent="swivel_link" xyz="0 0.05 0.02"/>
+  <xacro:head_joint name="head_left" xyz="0.03 0.03 0.05"/>
+  <xacro:head_joint name="head_right" xyz="-0.03 0.03 0.05"/>
+  <!-- Face screen mount -->
+  <link name="face_frame_link">
+    <visual>
+      <geometry><box size="0.08 0.02 0.06"/></geometry>
+      <origin xyz="0 0.06 0.1" rpy="0 0 0"/>
+      <material name="blue"><color rgba="0.2 0.4 0.9 1.0"/></material>
+    </visual>
+  </link>
+  <joint name="face_mount" type="fixed">
+    <parent link="base_joint_link"/>
+    <child link="face_frame_link"/>
+    <origin xyz="0 0.05 0.1" rpy="0 0 0"/>
+  </joint>
 </robot>
